File: NUCLEO-F401RE/NFC/kicad/ant7_t_st25dv04k.kicad_pcb (KiCad board)
At the start: 2 copper layers, 9 parts, among them J1 Conn_01x08_Male, J2 Conn_01x06_Male, J3 Conn_01x05_Male, J4 Conn_01x10_Male, J5 Conn_01x08_Male, U1 tactile_sw

Commit message: schematic update
Parts:
- added D1: LED GREEN, mcu:LED, F.Cu at (137.2, 109.2)
- added D2: LED BLUE, mcu:LED, F.Cu at (137.2, 114.3)
- added D3: LED RED, mcu:LED, F.Cu at (137.2, 119.4)
- added R4: 51k, mcu:Register, F.Cu at (147.3, 121.9)
- added R5: 51k, mcu:Register, F.Cu at (147.3, 124.5)
- added R6: 10k, mcu:Register, F.Cu at (147.3, 129.5)
- moved R1 9.92 mm to (125.7, 102.9)
- moved R2 9.92 mm to (128.3, 102.9)
- moved R3 9.92 mm to (123.2, 102.9)
- moved J3 6.35 mm to (128.3, 132.1)
Routing:
- net GND: track 72.4 -> 105.4 mm
- net Net-(J3-Pad5): track 78.7 -> 97.8 mm
- net Net-(D1-Pad2): track 0.00 -> 17.8 mm
- net Net-(D3-Pad2): track 0.00 -> 15.2 mm
- net Net-(D2-Pad2): track 0.00 -> 15.2 mm
- net Net-(J3-Pad4): track 63.5 -> 69.9 mm
- net Net-(J3-Pad3): track 63.5 -> 69.8 mm
- net +3V3: track 55.9 -> 62.2 mm
- net Net-(J5-Pad6): track 0.00 -> 3.81 mm
- net Net-(J5-Pad4): track 0.00 -> 3.81 mm
- net Net-(J5-Pad3): track 0.00 -> 3.81 mm

Commit message: update
Parts:
- moved D1 10.2 mm to (137.2, 99.1)
- moved D2 10.2 mm to (137.2, 104.1)
- moved D3 10.2 mm to (137.2, 109.2)
Routing:
- net Net-(D3-Pad2): track 15.2 -> 25.4 mm
- net Net-(D2-Pad2): track 15.2 -> 25.4 mm
- net Net-(D1-Pad2): track 17.8 -> 27.9 mm
- net GND: track 105.4 -> 115.6 mm
- net Net-(J3-Pad5): track 97.8 -> 92.7 mm
- net +3V3: track 62.2 -> 57.2 mm
